Commit message: use xacro to generate urdf for spot

File: dcist_launch_system/urdf/accessories.urdf.xacro (robot description, xacro)
@@ -10,15 +10,15 @@
       <visual>
         <geometry>
-          <mesh filename="package://spot_description/meshes/base/visual/pack_top.obj"/>
+          <mesh filename="package://dcist_launch_system/meshes/base/visual/pack_top.obj"/>
         </geometry>
       </visual>
       <visual>
         <geometry>
-          <mesh filename="package://spot_description/meshes/base/visual/pack_body.obj"/>
+          <mesh filename="package://dcist_launch_system/meshes/base/visual/pack_body.obj"/>
         </geometry>
       </visual>
       <collision>
         <geometry>
-          <mesh filename="package://spot_description/meshes/base/visual/pack_body.obj"/>
+          <mesh filename="package://dcist_launch_system/meshes/base/visual/pack_body.obj"/>
         </geometry>
       </collision>
@@ -34,10 +34,10 @@
       <visual>
         <geometry>
-          <mesh filename="package://spot_description/meshes/base/visual/lidar_mount.obj"/>
+          <mesh filename="package://dcist_launch_system/meshes/base/visual/lidar_mount.obj"/>
         </geometry>
       </visual>
       <collision>
         <geometry>
-          <mesh filename="package://spot_description/meshes/base/collision/lidar_mount_collision.stl"/>
+          <mesh filename="package://dcist_launch_system/meshes/base/collision/lidar_mount_collision.stl"/>
         </geometry>
       </collision>
@@ -53,5 +53,5 @@
         <visual>
           <geometry>
-            <mesh filename="package://spot_description/meshes/base/collision/velodyne_cage.stl" scale="0.001 0.001 0.001" />
+            <mesh filename="package://dcist_launch_system/meshes/base/collision/velodyne_cage.stl" scale="0.001 0.001 0.001" />
           </geometry>
           <origin xyz="0 0 0" rpy="0 0 0" />
@@ -60,5 +60,5 @@
         <collision>
           <geometry>
-            <mesh filename="package://spot_description/meshes/base/collision/velodyne_cage.stl" scale="0.001 0.001 0.001" />
+            <mesh filename="package://dcist_launch_system/meshes/base/collision/velodyne_cage.stl" scale="0.001 0.001 0.001" />
           </geometry>
           <origin xyz="0 0 0" rpy="0 0 0" />

File: dcist_launch_system/urdf/spot.urdf.xacro (robot description, xacro)
@@ -2,7 +2,7 @@
 <robot name="spot" xmlns:xacro="http://www.ros.org/wiki/xacro">
   <!-- Macro for loading Spot -->
-  <xacro:include filename="$(find spot_description)/urdf/spot_macro.xacro" />
+  <xacro:include filename="$(find dcist_launch_system)/urdf/spot_macro.xacro" />
   <!-- Macros for loading the ROS 2 control tags -->
-  <xacro:include filename="$(find spot_description)/urdf/spot.ros2_control.xacro" />
+  <xacro:include filename="$(find dcist_launch_system)/urdf/spot.ros2_control.xacro" />
   <!-- General parameters -->
   <!-- String that will be prepended to all joints and links-->

File: dcist_launch_system/urdf/spot_macro.xacro (robot description, xacro)
@@ -11,11 +11,11 @@
             <visual>
                 <geometry>
-                    <mesh filename="package://spot_description/meshes/base/visual/body.obj" />
-                </geometry>
-            </visual>
-            <collision>
-                <geometry>
-                    <mesh
-                        filename="package://spot_description/meshes/base/collision/body_collision.obj" />
+                    <mesh filename="package://dcist_launch_system/meshes/base/visual/body.obj" />
+                </geometry>
+            </visual>
+            <collision>
+                <geometry>
+                    <mesh
+                        filename="package://dcist_launch_system/meshes/base/collision/body_collision.obj" />
                 </geometry>
             </collision>
@@ -63,5 +63,5 @@
                 <geometry>
                     <mesh
-                        filename="package://spot_description/meshes/base/visual/front_left_hip.obj" />
+                        filename="package://dcist_launch_system/meshes/base/visual/front_left_hip.obj" />
                 </geometry>
             </visual>
@@ -97,11 +97,11 @@
                 <geometry>
                     <mesh
-                        filename="package://spot_description/meshes/base/visual/front_left_upper_leg.obj" />
-                </geometry>
-            </visual>
-            <collision>
-                <geometry>
-                    <mesh
-                        filename="package://spot_description/meshes/base/collision/left_upper_leg_collision.obj" />
+                        filename="package://dcist_launch_system/meshes/base/visual/front_left_upper_leg.obj" />
+                </geometry>
+            </visual>
+            <collision>
+                <geometry>
+                    <mesh
+                        filename="package://dcist_launch_system/meshes/base/collision/left_upper_leg_collision.obj" />
                 </geometry>
             </collision>
@@ -137,11 +137,11 @@
                 <geometry>
                     <mesh
-                        filename="package://spot_description/meshes/base/visual/front_left_lower_leg.obj" />
-                </geometry>
-            </visual>
-            <collision>
-                <geometry>
-                    <mesh
-                        filename="package://spot_description/meshes/base/collision/left_lower_leg_collision.obj" />
+                        filename="package://dcist_launch_system/meshes/base/visual/front_left_lower_leg.obj" />
+                </geometry>
+            </visual>
+            <collision>
+                <geometry>
+                    <mesh
+                        filename="package://dcist_launch_system/meshes/base/collision/left_lower_leg_collision.obj" />
                 </geometry>
             </collision>
@@ -183,5 +183,5 @@
                 <geometry>
                     <mesh
-                        filename="package://spot_description/meshes/base/visual/front_right_hip.obj" />
+                        filename="package://dcist_launch_system/meshes/base/visual/front_right_hip.obj" />
                 </geometry>
             </visual>
@@ -217,11 +217,11 @@
                 <geometry>
                     <mesh
-                        filename="package://spot_description/meshes/base/visual/front_right_upper_leg.obj" />
-                </geometry>
-            </visual>
-            <collision>
-                <geometry>
-                    <mesh
-                        filename="package://spot_description/meshes/base/collision/right_upper_leg_collision.obj" />
+                        filename="package://dcist_launch_system/meshes/base/visual/front_right_upper_leg.obj" />
+                </geometry>
+            </visual>
+            <collision>
+                <geometry>
+                    <mesh
+                        filename="package://dcist_launch_system/meshes/base/collision/right_upper_leg_collision.obj" />
                 </geometry>
             </collision>
@@ -257,11 +257,11 @@
                 <geometry>
                     <mesh
-                        filename="package://spot_description/meshes/base/visual/front_right_lower_leg.obj" />
-                </geometry>
-            </visual>
-            <collision>
-                <geometry>
-                    <mesh
-                        filename="package://spot_description/meshes/base/collision/right_lower_leg_collision.obj" />
+                        filename="package://dcist_launch_system/meshes/base/visual/front_right_lower_leg.obj" />
+                </geometry>
+            </visual>
+            <collision>
+                <geometry>
+                    <mesh
+                        filename="package://dcist_launch_system/meshes/base/collision/right_lower_leg_collision.obj" />
                 </geometry>
             </collision>
@@ -303,5 +303,5 @@
                 <geometry>
                     <mesh
-                        filename="package://spot_description/meshes/base/visual/rear_left_hip.obj" />
+                        filename="package://dcist_launch_system/meshes/base/visual/rear_left_hip.obj" />
                 </geometry>
             </visual>
@@ -337,11 +337,11 @@
                 <geometry>
                     <mesh
-                        filename="package://spot_description/meshes/base/visual/rear_left_upper_leg.obj" />
-                </geometry>
-            </visual>
-            <collision>
-                <geometry>
-                    <mesh
-                        filename="package://spot_description/meshes/base/collision/left_upper_leg_collision.obj" />
+                        filename="package://dcist_launch_system/meshes/base/visual/rear_left_upper_leg.obj" />
+                </geometry>
+            </visual>
+            <collision>
+                <geometry>
+                    <mesh
+                        filename="package://dcist_launch_system/meshes/base/collision/left_upper_leg_collision.obj" />
                 </geometry>
             </collision>
@@ -377,11 +377,11 @@
                 <geometry>
                     <mesh
-                        filename="package://spot_description/meshes/base/visual/rear_left_lower_leg.obj" />
-                </geometry>
-            </visual>
-            <collision>
-                <geometry>
-                    <mesh
-                        filename="package://spot_description/meshes/base/collision/left_lower_leg_collision.obj" />
+                        filename="package://dcist_launch_system/meshes/base/visual/rear_left_lower_leg.obj" />
+                </geometry>
+            </visual>
+            <collision>
+                <geometry>
+                    <mesh
+                        filename="package://dcist_launch_system/meshes/base/collision/left_lower_leg_collision.obj" />
                 </geometry>
             </collision>
@@ -423,5 +423,5 @@
                 <geometry>
                     <mesh
-                        filename="package://spot_description/meshes/base/visual/rear_right_hip.obj" />
+                        filename="package://dcist_launch_system/meshes/base/visual/rear_right_hip.obj" />
                 </geometry>
             </visual>
@@ -457,11 +457,11 @@
                 <geometry>
                     <mesh
-                        filename="package://spot_description/meshes/base/visual/rear_right_upper_leg.obj" />
-                </geometry>
-            </visual>
-            <collision>
-                <geometry>
-                    <mesh
-                        filename="package://spot_description/meshes/base/collision/right_upper_leg_collision.obj" />
+                        filename="package://dcist_launch_system/meshes/base/visual/rear_right_upper_leg.obj" />
+                </geometry>
+            </visual>
+            <collision>
+                <geometry>
+                    <mesh
+                        filename="package://dcist_launch_system/meshes/base/collision/right_upper_leg_collision.obj" />
                 </geometry>
             </collision>
@@ -497,11 +497,11 @@
                 <geometry>
                     <mesh
-                        filename="package://spot_description/meshes/base/visual/rear_right_lower_leg.obj" />
-                </geometry>
-            </visual>
-            <collision>
-                <geometry>
-                    <mesh
-                        filename="package://spot_description/meshes/base/collision/right_lower_leg_collision.obj" />
+                        filename="package://dcist_launch_system/meshes/base/visual/rear_right_lower_leg.obj" />
+                </geometry>
+            </visual>
+            <collision>
+                <geometry>
+                    <mesh
+                        filename="package://dcist_launch_system/meshes/base/collision/right_lower_leg_collision.obj" />
                 </geometry>
             </collision>
@@ -540,11 +540,11 @@
         </xacro:if>
         <!-- Standard accessories. -->
-        <xacro:include filename="$(find spot_description)/urdf/accessories.urdf.xacro" />
+        <xacro:include filename="$(find dcist_launch_system)/urdf/accessories.urdf.xacro" />
         <!-- Optional custom includes. -->
-        <xacro:property name="default_empty_urdf" value="$(find spot_description)/urdf/empty.urdf" />
+        <xacro:property name="default_empty_urdf" value="$(find dcist_launch_system)/urdf/empty.urdf" />
         <xacro:include filename="$(optenv SPOT_URDF_EXTRAS ${default_empty_urdf})" />
         <!-- Include Arm if necessary-->
         <xacro:if value="${arm}">
-            <xacro:include filename="$(find spot_description)/urdf/spot_arm_macro.urdf" />
+            <xacro:include filename="$(find dcist_launch_system)/urdf/spot_arm_macro.urdf" />
             <xacro:load_arm tf_prefix="${tf_prefix}"
                             gripperless="${gripperless}"
@@ -553,5 +553,5 @@
         <!-- Include links at feet if necessary -->
         <xacro:if value="${feet}">
-            <xacro:include filename="$(find spot_description)/urdf/spot_feet_macro.urdf" />
+            <xacro:include filename="$(find dcist_launch_system)/urdf/spot_feet_macro.urdf" />
             <xacro:load_feet tf_prefix="${tf_prefix}" />
         </xacro:if>

File: dcist_launch_system/urdf/spot_simple.urdf.xacro (robot description, xacro)
@@ -5,5 +5,5 @@
       <origin xyz="0 0 0" rpy="0 0 0"/>
       <geometry>
-        <mesh filename="package://spot_description/meshes/base_simple/visual/body.obj"/>
+        <mesh filename="package://dcist_launch_system/meshes/base_simple/visual/body.obj"/>
       </geometry>
       <material name="body"> <color rgba="1 0.8431 0 1"/></material>
@@ -11,5 +11,5 @@
     <collision>
       <geometry>
-        <mesh filename="package://spot_description/meshes/base_simple/collision/body.stl" />
+        <mesh filename="package://dcist_launch_system/meshes/base_simple/collision/body.stl" />
       </geometry>
     </collision>
@@ -31,5 +31,5 @@
       <origin xyz="0 0 0" rpy="0 0 0"/>
       <geometry>
-        <mesh filename="package://spot_description/meshes/base_simple/visual/fl_hip.obj"/>
+        <mesh filename="package://dcist_launch_system/meshes/base_simple/visual/fl_hip.obj"/>
       </geometry>
       <material name="fl_hip"> <color rgba="0.2 0.2 0.2 1"/></material>
@@ -37,5 +37,5 @@
     <collision>
       <geometry>
-        <mesh filename="package://spot_description/meshes/base_simple/collision/fl_hip.stl" />
+        <mesh filename="package://dcist_launch_system/meshes/base_simple/collision/fl_hip.stl" />
       </geometry>
     </collision>
@@ -57,5 +57,5 @@
       <origin xyz="0 0 0" rpy="0 0 0"/>
       <geometry>
-        <mesh filename="package://spot_description/meshes/base_simple/visual/fl_uleg.obj"/>
+        <mesh filename="package://dcist_launch_system/meshes/base_simple/visual/fl_uleg.obj"/>
       </geometry>
       <material name="fl_uleg"> <color rgba="1 0.8431 0 1"/></material>
@@ -63,5 +63,5 @@
     <collision>
       <geometry>
-        <mesh filename="package://spot_description/meshes/base_simple/collision/fl_uleg.stl" />
+        <mesh filename="package://dcist_launch_system/meshes/base_simple/collision/fl_uleg.stl" />
       </geometry>
     </collision>
@@ -83,5 +83,5 @@
       <origin xyz="0 0 0" rpy="0 0 0"/>
       <geometry>
-        <mesh filename="package://spot_description/meshes/base_simple/visual/fl_lleg.obj"/>
+        <mesh filename="package://dcist_launch_system/meshes/base_simple/visual/fl_lleg.obj"/>
       </geometry>
       <material name="fl_lleg"> <color rgba="0.2 0.2 0.2 1"/></material>
@@ -89,5 +89,5 @@
     <collision>
       <geometry>
-        <mesh filename="package://spot_description/meshes/base_simple/collision/fl_lleg.stl" />
+        <mesh filename="package://dcist_launch_system/meshes/base_simple/collision/fl_lleg.stl" />
       </geometry>
     </collision>
@@ -109,5 +109,5 @@
       <origin xyz="0 0 0" rpy="0 0 0"/>
       <geometry>
-        <mesh filename="package://spot_description/meshes/base_simple/visual/fr_hip.obj"/>
+        <mesh filename="package://dcist_launch_system/meshes/base_simple/visual/fr_hip.obj"/>
       </geometry>
       <material name="fr_hip"> <color rgba="0.2 0.2 0.2 1"/></material>
@@ -115,5 +115,5 @@
     <collision>
       <geometry>
-        <mesh filename="package://spot_description/meshes/base_simple/collision/fr_hip.stl" />
+        <mesh filename="package://dcist_launch_system/meshes/base_simple/collision/fr_hip.stl" />
       </geometry>
     </collision>
@@ -135,5 +135,5 @@
       <origin xyz="0 0 0" rpy="0 0 0"/>
       <geometry>
-        <mesh filename="package://spot_description/meshes/base_simple/visual/fr_uleg.obj"/>
+        <mesh filename="package://dcist_launch_system/meshes/base_simple/visual/fr_uleg.obj"/>
       </geometry>
       <material name="fr_uleg"> <color rgba="1 0.8431 0 1"/></material>
@@ -141,5 +141,5 @@
     <collision>
       <geometry>
-        <mesh filename="package://spot_description/meshes/base_simple/collision/fr_uleg.stl" />
+        <mesh filename="package://dcist_launch_system/meshes/base_simple/collision/fr_uleg.stl" />
       </geometry>
     </collision>
@@ -161,5 +161,5 @@
       <origin xyz="0 0 0" rpy="0 0 0"/>
       <geometry>
-        <mesh filename="package://spot_description/meshes/base_simple/visual/fr_lleg.obj"/>
+        <mesh filename="package://dcist_launch_system/meshes/base_simple/visual/fr_lleg.obj"/>
       </geometry>
       <material name="fr_lleg"> <color rgba="0.2 0.2 0.2 1"/></material>
@@ -167,5 +167,5 @@
     <collision>
       <geometry>
-        <mesh filename="package://spot_description/meshes/base_simple/collision/fr_lleg.stl" />
+        <mesh filename="package://dcist_launch_system/meshes/base_simple/collision/fr_lleg.stl" />
       </geometry>
     </collision>
@@ -187,5 +187,5 @@
       <origin xyz="0 0 0" rpy="0 0 0"/>
       <geometry>
-        <mesh filename="package://spot_description/meshes/base_simple/visual/hl_hip.obj"/>
+        <mesh filename="package://dcist_launch_system/meshes/base_simple/visual/hl_hip.obj"/>
       </geometry>
       <material name="hl_hip"> <color rgba="0.2 0.2 0.2 1"/></material>
@@ -193,5 +193,5 @@
     <collision>
       <geometry>
-        <mesh filename="package://spot_description/meshes/base_simple/collision/hl_hip.stl" />
+        <mesh filename="package://dcist_launch_system/meshes/base_simple/collision/hl_hip.stl" />
       </geometry>
     </collision>
@@ -213,5 +213,5 @@
       <origin xyz="0 0 0" rpy="0 0 0"/>
       <geometry>
-        <mesh filename="package://spot_description/meshes/base_simple/visual/hl_uleg.obj"/>
+        <mesh filename="package://dcist_launch_system/meshes/base_simple/visual/hl_uleg.obj"/>
       </geometry>
       <material name="hl_uleg"> <color rgba="1 0.8431 0 1"/></material>
@@ -219,5 +219,5 @@
     <collision>
       <geometry>
-        <mesh filename="package://spot_description/meshes/base_simple/collision/hl_uleg.stl" />
+        <mesh filename="package://dcist_launch_system/meshes/base_simple/collision/hl_uleg.stl" />
       </geometry>
     </collision>
@@ -239,5 +239,5 @@
       <origin xyz="0 0 0" rpy="0 0 0"/>
       <geometry>
-        <mesh filename="package://spot_description/meshes/base_simple/visual/hl_lleg.obj"/>
+        <mesh filename="package://dcist_launch_system/meshes/base_simple/visual/hl_lleg.obj"/>
       </geometry>
       <material name="hl_lleg"> <color rgba="0.2 0.2 0.2 1"/></material>
@@ -245,5 +245,5 @@
     <collision>
       <geometry>
-        <mesh filename="package://spot_description/meshes/base_simple/collision/hl_lleg.stl" />
+        <mesh filename="package://dcist_launch_system/meshes/base_simple/collision/hl_lleg.stl" />
       </geometry>
     </collision>
@@ -265,5 +265,5 @@
       <origin xyz="0 0 0" rpy="0 0 0"/>
       <geometry>
-        <mesh filename="package://spot_description/meshes/base_simple/visual/hr_hip.obj"/>
+        <mesh filename="package://dcist_launch_system/meshes/base_simple/visual/hr_hip.obj"/>
       </geometry>
       <material name="hr_hip"> <color rgba="0.2 0.2 0.2 1"/></material>
@@ -271,5 +271,5 @@
     <collision>
       <geometry>
-        <mesh filename="package://spot_description/meshes/base_simple/collision/hr_hip.stl" />
+        <mesh filename="package://dcist_launch_system/meshes/base_simple/collision/hr_hip.stl" />
       </geometry>
     </collision>
@@ -291,5 +291,5 @@
       <origin xyz="0 0 0" rpy="0 0 0"/>
       <geometry>
-        <mesh filename="package://spot_description/meshes/base_simple/visual/hr_uleg.obj"/>
+        <mesh filename="package://dcist_launch_system/meshes/base_simple/visual/hr_uleg.obj"/>
       </geometry>
       <material name="hr_uleg"> <color rgba="1 0.8431 0 1"/></material>
@@ -297,5 +297,5 @@
     <collision>
       <geometry>
-        <mesh filename="package://spot_description/meshes/base_simple/collision/hr_uleg.stl" />
+        <mesh filename="package://dcist_launch_system/meshes/base_simple/collision/hr_uleg.stl" />
       </geometry>
     </collision>
@@ -317,5 +317,5 @@
       <origin xyz="0 0 0" rpy="0 0 0"/>
       <geometry>
-        <mesh filename="package://spot_description/meshes/base_simple/visual/hr_lleg.obj"/>
+        <mesh filename="package://dcist_launch_system/meshes/base_simple/visual/hr_lleg.obj"/>
       </geometry>
       <material name="hr_lleg"> <color rgba="0.2 0.2 0.2 1"/></material>
@@ -323,5 +323,5 @@
     <collision>
       <geometry>
-        <mesh filename="package://spot_description/meshes/base_simple/collision/hr_lleg.stl" />
+        <mesh filename="package://dcist_launch_system/meshes/base_simple/collision/hr_lleg.stl" />
       </geometry>
     </collision>
@@ -340,5 +340,5 @@
   </joint>
   <!-- Standard accessories. -->
-  <!-- <xacro:include filename="$(find spot_description)/urdf/accessories.urdf.xacro" /> -->
+  <!-- <xacro:include filename="$(find dcist_launch_system)/urdf/accessories.urdf.xacro" /> -->
   <!-- Optional custom includes. -->
   <!-- <xacro:include filename="$(optenv SPOT_URDF_EXTRAS empty.urdf)" /> -->

File: dcist_launch_system/urdf/standalone_arm.urdf.xacro (robot description, xacro)
@@ -1,5 +1,5 @@
 <?xml version="1.0"?>
 <robot name="standalone_arm" xmlns:xacro="http://www.ros.org/wiki/xacro">
-  <xacro:include filename="$(find spot_description)/urdf/spot_arm_macro.urdf" />
+  <xacro:include filename="$(find dcist_launch_system)/urdf/spot_arm_macro.urdf" />
   <!-- Root link -->
   <link name="body"/>

File: dcist_launch_system/urdf/standalone_gripper.urdf.xacro (robot description, xacro)
@@ -1,5 +1,5 @@
 <?xml version="1.0"?>
 <robot name="standalone_gripper" xmlns:xacro="http://www.ros.org/wiki/xacro">
-  <xacro:include filename="$(find spot_description)/urdf/spot_gripper_macro.urdf" />
+  <xacro:include filename="$(find dcist_launch_system)/urdf/spot_gripper_macro.urdf" />
   <!-- Root link -->
   <!-- <link name="body"/> -->
