Commit message: system working using zed2i camera
- update roman / roman_ros
- update roman config files (using Dino now, give yolo weights path)
- add roman loop closure visualization
- update hydra config to work with zed
- update hydra launch
- add yolo weights downloading in install
- update topaz camera calibration

File: dcist_launch_system/urdf/topaz.urdf.xacro (robot description, xacro)
@@ -11,5 +11,5 @@
     <parent link="$(arg tf_prefix)/frontleft"/>
     <child link="$(arg tf_prefix)_zed_camera_link"/>
-    <origin xyz="-0.10658496884512007 0.026247948174877016 -0.11793444318564054" rpy="-2.6228496639972296 1.3036971096950234 3.1196051589865026" />
+    <origin xyz="-0.14202953085743672 0.015046794634271764 0.07455903427663088" rpy="-1.990205509681296 -0.972943029332566 2.0587233433215095" />
   </joint>
 </robot>

Commit message: update topaz camera calibration and add spot recording scripts

File: dcist_launch_system/urdf/topaz.urdf.xacro (robot description, xacro)
@@ -11,5 +11,5 @@
     <parent link="$(arg tf_prefix)/frontleft"/>
     <child link="$(arg tf_prefix)_zed_camera_link"/>
-    <origin xyz="-0.14202953085743672 0.015046794634271764 0.07455903427663088" rpy="-1.990205509681296 -0.972943029332566 2.0587233433215095" />
+    <origin xyz="-0.1377625424350767 0.021380403878896944 0.057657655316766976" rpy="-2.004012441564318 -0.9950601951115012 2.083327840660515" />
   </joint>
 </robot>
